File: AgroNeck.kicad_pcb (KiCad board)
At the start: 2 copper layers, 24 parts, among them J1 Screw_Terminal_01x02, J2 CONTROLVCC, U6 LM35-LP, U7 LM358

Commit message: last version(incomplete)
Parts:
- removed C1, C3: 100nf, Capacitor_THT:CP_Radial_D8.0mm_P5.00mm
- removed C2: 2.2nF or 1nF, Capacitor_THT:CP_Radial_D8.0mm_P5.00mm
- removed R1: 470k, Resistor_THT:R_Axial_DIN0309_L9.0mm_D3.2mm_P15.24mm_Horizontal
- removed R2: 1M, Resistor_THT:R_Axial_DIN0309_L9.0mm_D3.2mm_P15.24mm_Horizontal
- removed R3, R4: 100k, Resistor_THT:R_Axial_DIN0309_L9.0mm_D3.2mm_P15.24mm_Horizontal
- removed R5, R7: 10k, Resistor_THT:R_Axial_DIN0309_L9.0mm_D3.2mm_P15.24mm_Horizontal
- removed R6: 1k, Resistor_THT:R_Axial_DIN0309_L9.0mm_D3.2mm_P15.24mm_Horizontal
- removed U4: ~, Connector_PinSocket_2.54mm:PinSocket_1x08_P2.54mm_Vertical
- removed U7: LM358, Package_DIP:DIP-8_W10.16mm_LongPads
- added J3: Screw_Terminal_01x04, TerminalBlock:TerminalBlock_MaiXu_MX126-5.0-04P_1x04_P5.00mm, F.Cu at (166.5, 119.5)
- J1: value Screw_Terminal_01x02 -> Screw_Terminal_01x08; footprint TerminalBlock:TerminalBlock_MaiXu_MX126-5.0-02P_1x02_P5.00mm -> Connector_PinHeader_2.54mm:PinHeader_1x08_P2.54mm_Vertical
- moved C6 107.2 mm to (171.7, 72.5), turned to 180 degrees
- moved C7 105.7 mm to (172.0, 92.0), turned to 180 degrees
- moved C8 104.9 mm to (172.0, 82.5), turned to 180 degrees
- moved C4 65.1 mm to (203.0, 103.0)
- moved U3 54.5 mm to (174.8, 28.1), turned to 90 degrees
- moved U2 40.6 mm to (118.0, 44.3)
- moved J2 37.7 mm to (149.5, 130.9)
- moved J1 37.4 mm to (85.0, 87.7), turned to 180 degrees
- moved U5 34.3 mm to (185.0, 85.0)
- moved U6 31.1 mm to (92.0, 45.0)
- moved C5 27.4 mm to (158.0, 95.0)
- moved U8 25.5 mm to (97.4, 87.8)
Connections:
- J1 pad 2: PIEZOELECTRICO_IN -> VCC
Routing:
- net LORA_MISO: track 0.00 -> 70.2 mm
- net LORA_MOSI: track 0.00 -> 68.4 mm
- net Net-(U7A-+): track 63.6 -> 0.00 mm
- net Net-(C2-Pad1): track 59.0 -> 0.00 mm
- net Net-(U7A--): track 55.1 -> 0.00 mm
- net LORA_CLK: track 0.00 -> 51.2 mm
- net LORA_CS: track 0.00 -> 47.6 mm
- net +3V3: track 60.0 -> 19.7 mm
- net MLX_MPU6050_SCL: track 0.00 -> 36.9 mm
- net MLX_MPU6050_SDA: track 0.00 -> 34.8 mm
- net VCC: track 0.00 -> 32.6 mm
- net GND: track 83.4 -> 58.1 mm
- net Net-(C1-Pad2): track 9.57 -> 0.00 mm
Other:
- board outline added: 120 x 120 mm
