File: AgroNeck.kicad_sch (KiCad schematic)
At the start: 22 parts, among them U6 LM35-LP, U7 LM358

Commit message: actulizado sin pcb
Parts:
- removed U1: (no value), symbol My_esp32:ESP32_Devkit_1
- added J1: Screw_Terminal_01x02, TerminalBlock:TerminalBlock_MaiXu_MX126-5.0-02P_1x02_P5.00mm, symbol Connector:Screw_Terminal_01x02
- added J2: CONTROLVCC, TerminalBlock:TerminalBlock_MaiXu_MX126-5.0-06P_1x06_P5.00mm, symbol Connector:Screw_Terminal_01x06
- added U8: (no value), ESP32:ESP32_devkit1, symbol ESP32_devkit_38P:esp32_1
- C1, C2, C3, C4, C5, C6, C7, C8: footprint (none) -> Capacitor_THT:CP_Radial_D8.0mm_P5.00mm
- R1, R2, R3, R4, R5, R6, R7: footprint (none) -> Resistor_THT:R_Axial_DIN0309_L9.0mm_D3.2mm_P15.24mm_Horizontal
- U2: footprint (none) -> MPU:MPU6050
- U3: footprint (none) -> GPS:GY-NEO6MV2
- U4: footprint (none) -> Connector_PinSocket_2.54mm:PinSocket_1x08_P2.54mm_Vertical
- U5: footprint (none) -> TerminalBlock:TerminalBlock_MaiXu_MX126-5.0-04P_1x04_P5.00mm
- U7: footprint (none) -> Package_DIP:DIP-8_W10.16mm_LongPads
Connections:
- net +3V3: now also U8.1 (3.3V)
- net GND: now also J1.1 (Pin_1), J2.6 (Pin_6), U8.14 (GND), U8.20 (GND), U8.26 (GND)
- net LORA_CLK: now also U8.28 (GPIO18)
- net LORA_CS: now also U8.29 (GPIO5)
- net LORA_DIO0: now also U8.17 (GPIO13)
- net LORA_MISO: now also U8.27 (GPIO19)
- net LORA_MOSI: now also U8.21 (GPIO23)
- net LORA_RESET: now also U8.12 (GPIO14)
- net MLX_MPU6050_SCL: now also U8.22 (GPIO22)
- net MLX_MPU6050_SDA: now also U8.25 (GPIO21)
- net MPU6050_INT: now also U8.11 (GPIO27)
- net NEO6M_RX: now also U8.31 (GPIO16)
- net NEO6M_TX: now also U8.30 (GPIO17)
- net PIEZOELECTRICO_IN: now also J1.2 (Pin_2)
- net PIEZOELECTRICO_OUT: now also U8.6 (GPIO35)
- net VCC: now also J2.5 (Pin_5), U8.19 (VIN)
- net V_LM35: now also U8.5 (GPIO34)
- net at C5.2: now also U8.2 (EN)
- new net CONTROL1: J2.1 (Pin_1), U8.7 (GPIO32)
- new net CONTROL2: J2.2 (Pin_2), U8.8 (GPIO33)
- new net CONTROL3: J2.3 (Pin_3), U8.9 (GPIO25)
- new net CONTROL4: J2.4 (Pin_4), U8.10 (GPIO26)
Other:
- moved on the sheet: C5

Commit message: last version(incomplete)
Parts:
- removed C1, C3: 100nf, Capacitor_THT:CP_Radial_D8.0mm_P5.00mm, symbol Device:C_Small
- removed C2: 2.2nF or 1nF, Capacitor_THT:CP_Radial_D8.0mm_P5.00mm, symbol Device:C_Small
- removed J1: Screw_Terminal_01x02, TerminalBlock:TerminalBlock_MaiXu_MX126-5.0-02P_1x02_P5.00mm, symbol Connector:Screw_Terminal_01x02
- removed R1: 470k, Resistor_THT:R_Axial_DIN0309_L9.0mm_D3.2mm_P15.24mm_Horizontal, symbol Device:R
- removed R2: 1M, Resistor_THT:R_Axial_DIN0309_L9.0mm_D3.2mm_P15.24mm_Horizontal, symbol Device:R
- removed R3, R4: 100k, Resistor_THT:R_Axial_DIN0309_L9.0mm_D3.2mm_P15.24mm_Horizontal, symbol Device:R
- removed R5, R7: 10k, Resistor_THT:R_Axial_DIN0309_L9.0mm_D3.2mm_P15.24mm_Horizontal, symbol Device:R
- removed R6: 1k, Resistor_THT:R_Axial_DIN0309_L9.0mm_D3.2mm_P15.24mm_Horizontal, symbol Device:R
- removed U4: (no value), Connector_PinSocket_2.54mm:PinSocket_1x08_P2.54mm_Vertical, symbol LORA_Xl1278:Xl1278-smt
- removed U7: LM358, Package_DIP:DIP-8_W10.16mm_LongPads, symbol Amplifier_Operational:LM358
- added J1: Screw_Terminal_01x08, Connector_PinHeader_2.54mm:PinHeader_1x08_P2.54mm_Vertical, symbol Connector:Screw_Terminal_01x08
- added J3: Screw_Terminal_01x04, TerminalBlock:TerminalBlock_MaiXu_MX126-5.0-04P_1x04_P5.00mm, symbol Connector:Screw_Terminal_01x04
Connections:
- net +3V3: now also J3.1 (Pin_1)
- net GND: now also J1.1 (Pin_1), J3.2 (Pin_2), J3.4 (Pin_4)
- net LORA_CLK: now also J1.5 (Pin_5)
- net LORA_CS: now also J1.6 (Pin_6)
- net LORA_DIO0: now also J1.7 (Pin_7)
- net LORA_MISO: now also J1.3 (Pin_3)
- net LORA_MOSI: now also J1.4 (Pin_4)
- net LORA_RESET: now also J1.8 (Pin_8)
- net PIEZOELECTRICO_OUT: now also J3.3 (Pin_3)
- net VCC: now also J1.2 (Pin_2)
Other:
- note removed: "Amplificador Sensor Piezoelectrico"
